Commit message: Scaffold Look Twice v5 embodied navigation and proxy manipulation
Freeze V5 design, dual contracts (cross_region + pick_proxy), synthetic
closed-loop episode, workspace claims, URDF arm proxy, motion acceptance
script, and unit tests. Genesis runtime remains staged for W7900D.

File: assets/robots/look_twice_skid_steer.urdf (robot description, URDF)
Before this commit: robot look_twice_skid_steer, 6 links, 5 joints
Links:
- added link arm_link, mass 0.6; collision box size=0.24 0.04 0.04; visual box size=0.24 0.04 0.04
- link base_link: mass 8.0 -> 10.0; geometry collision box size=0.42 0.32 0.14; visual box size=0.42 0.32 0.14
- link left_front_wheel: mass 0.35 -> 0.40; geometry collision cylinder length=0.05 radius=0.07; visual cylinder length=0.05 radius=0.07
- link left_rear_wheel: mass 0.35 -> 0.40; geometry collision cylinder length=0.05 radius=0.07; visual cylinder length=0.05 radius=0.07
- link right_front_wheel: mass 0.35 -> 0.40; geometry collision cylinder length=0.05 radius=0.07; visual cylinder length=0.05 radius=0.07
- link right_rear_wheel: mass 0.35 -> 0.40; geometry collision cylinder length=0.05 radius=0.07; visual cylinder length=0.05 radius=0.07
Joints:
- added joint arm_fixed: type fixed, parent base_link, child arm_link, origin xyz=0.15 0 0.05
- joint left_front_wheel_joint: limit effort=20 velocity=20 -> effort=30 velocity=25; origin xyz=0.12 0.17 -0.04 -> xyz=0.13 0.18 -0.05
- joint left_rear_wheel_joint: limit effort=20 velocity=20 -> effort=30 velocity=25; origin xyz=-0.12 0.17 -0.04 -> xyz=-0.13 0.18 -0.05
- joint right_front_wheel_joint: limit effort=20 velocity=20 -> effort=30 velocity=25; origin xyz=0.12 -0.17 -0.04 -> xyz=0.13 -0.18 -0.05
- joint right_rear_wheel_joint: limit effort=20 velocity=20 -> effort=30 velocity=25; origin xyz=-0.12 -0.17 -0.04 -> xyz=-0.13 -0.18 -0.05
